File: Hardware/KiCad/RetroLink.kicad_sch (KiCad schematic)
At the start: 90 parts, among them CON1 HSMM-A100-S00J1, IC1 TLV320AIC1110PBS, IC12 BQ24090DGQR, IC2 IIC 0x3A MAX7329AWE+T, IC3 BC846AW-7-F, IC6 MCP1642B-50I_MS, IC7 IIC 0x38 MAX7329AWE+T, IC8 MAX40200AUK+T, J10 SAMTEC-HMTSW-101-24-X-S-290, J11 SAMTEC-HMTSW-101-24-X-S-290, J12 SAMTEC-HMTSW-101-24-X-S-290, J2 95501-2641, J21 PJS008-2120-0, J28 SAMTEC-HMTSW-101-24-X-S-290, Q1 BSS138, Q2 BSS138, U1 Ag1170-S5, U3 IIC 0x3C DM-OLED096-636, U5 1043

Commit message: audio cutout fixes, number lookup, misc updates
Parts:
- added R6, R8: 22K, RESC2013X65N, symbol WCR0805-10KFI:WCR0805-10KFI
- added R7, R9: 10K, RESC2013X65N, symbol WCR0805-10KFI:WCR0805-10KFI
Connections:
- net GND: now also R7.2, R9.2
- net at C1.2: now also R8.2; no longer U1.10 (VOUT)
- net at U1.9 (VIN): now also R6.1, R7.1; no longer C8.2
- new net: C8.2, R6.2
- new net: R8.1, R9.1, U1.10 (VOUT)
Other:
- moved on the sheet: C1, C8

Commit message: fixes to audio levels and gpio outputs
Parts:
- removed R9: 10K, RESC2013X65N, symbol WCR0805-10KFI:WCR0805-10KFI
- added C15: 0.1uF, CAPC3216X229N, symbol 12063G106ZAT2A:12063G106ZAT2A
- added IC4: SN74AHCT125DR, SOIC127P600X175-14N, symbol SN74AHCT125DR:SN74AHCT125DR
- R6: value 22K -> 0K
- R7: value 10K -> 8.2K
- R8: value 22K -> 47K
Connections:
- net +5V: now also C15.1, IC4.10 (3~{OE}), IC4.13 (4~{OE}), IC4.14 (VCC)
- net GND: now also C15.2, IC4.1 (1~{OE}), IC4.12 (4A), IC4.4 (2~{OE}), IC4.7 (GND), IC4.9 (3A); no longer R7.2
- net GPIO_7: now also IC4.2 (1A); no longer U1.3 (F/R)
- net GPIO_8: now also IC4.5 (2A); no longer U1.4 (RM)
- net at R6.1, U1.9 (VIN): no longer R7.1
- net at C1.1, IC1.2 (MIC1P): now also R7.1
- net at C10.2, IC1.3 (MIC1N): now also R7.2
- new net SLIC_FR: IC4.3 (1Y), U1.3 (F/R)
- new net SLIC_RM: IC4.6 (2Y), U1.4 (RM)
